File: Ver2/Board/Board.kicad_pcb (KiCad board)
At the start: 2 copper layers, 96.5 x 114.6 mm, 88 parts, among them J1 Vin, J10 SonicGND, J11 Proximity2, J12 Proximity2, J13 Proximity2, J2 MotorPWR, J3 Reset_switch, J4 LED strip, J5 Servo1, J6 Servo2, J7 Estop, J8 Swiss Sonic cable, J9 Screw_Terminal_01x12, Q1 BSS138, Q2 BSS138, Q3 BSS138, Q4 BSS138, Q5 BSS138, Q6 A03401-Peters, Q7 BSS138, U1 AP2210-3.3V, U10 PC817, U11 PC817, U12 PC817, U13 PC817, U14 PC817, U2 V7805-1000, U4 INA219, U5 PC817, U6 PC817, U7 PC817, U8 LM358N_LTB, U9 PC817

Commit message: routing
Parts:
- removed the H2 at (191.5, 92.4)
- removed the H2 at (105.5, 92.4)
- added D1: 26v, Diode_THT:D_DO-15_P10.16mm_Horizontal, F.Cu at (152.9, 65.0)
- added F1: Polyfuse, Libs:LittleFuse_110F_24V, B.Cu at (183.4, 55.1)
- added F2: 100-300mA, Libs:LittleFuse_110F_24V, B.Cu at (172.4, 53.8)
- added H3: MountingHole, MountingHole:MountingHole_3.2mm_M3, F.Cu at (191.5, 92.4)
- added H4: MountingHole, MountingHole:MountingHole_3.2mm_M3, F.Cu at (105.5, 92.4)
- added R35: 2K, Resistor_SMD:R_0805_2012Metric_Pad1.15x1.40mm_HandSolder, F.Cu at (156.7, 52.8)
- added R36: 1K-2K, Resistor_SMD:R_0805_2012Metric_Pad1.15x1.40mm_HandSolder, B.Cu at (125.3, 41.3)
- added R37: 10K, Resistor_SMD:R_0805_2012Metric_Pad1.15x1.40mm_HandSolder, B.Cu at (150.5, 53.5)
- added R38: 100R, Resistor_SMD:R_0805_2012Metric_Pad1.15x1.40mm_HandSolder, F.Cu at (163.0, 105.9)
- added REL1: IM03GR, Libs:IM03GR, F.Cu at (171.7, 110.7)
- added REL2: IM03GR, Libs:IM03GR, F.Cu at (155.7, 110.7)
- added U15: PC817, Package_DIP:DIP-4_W7.62mm, F.Cu at (150.4, 49.4)
- added U3: Bluepill, Libs:Bluepill, F.Cu at (134.4, 87.9)
- C2, C3, D3, R10, R13, R14, R16, R17, R23, R25, R29, R30, R32, R9: moved to B.Cu
- J11, J12, J13, J5, J6: footprint TerminalBlock_Phoenix:TerminalBlock_Phoenix_MPT-0,5-3-2.54_1x03_P2.54mm_Horizontal -> Libs:MKDS1,3-3,81
- J7: footprint TerminalBlock_Phoenix:TerminalBlock_Phoenix_MPT-0,5-2-2.54_1x02_P2.54mm_Horizontal -> TerminalBlock:TerminalBlock_bornier-2_P5.08mm
- moved R17 154.9 mm to (111.0, 41.3), turned to 270 degrees
- moved R29 149.3 mm to (115.6, 135.6)
- moved R16 148.3 mm to (117.5, 53.5), turned to 270 degrees
- moved R14 147.8 mm to (114.8, 41.3), turned to 270 degrees
- moved R27 147.7 mm to (115.7, 119.3), turned to 270 degrees
- moved R25 142.8 mm to (118.2, 41.3), turned to 270 degrees
- moved R30 142.2 mm to (127.8, 135.7)
- moved R28 138.9 mm to (127.2, 119.3), turned to 270 degrees
- moved R23 133.3 mm to (133.4, 53.5), turned to 270 degrees
- moved R13 129.7 mm to (125.4, 53.6), turned to 270 degrees
- moved R2 121.2 mm to (117.6, 81.4)
- moved R10 119.3 mm to (121.7, 41.3), turned to 270 degrees
- moved U6 118.7 mm to (125.3, 49.4), turned to 270 degrees
- moved R9 115.2 mm to (142.2, 53.5), turned to 270 degrees
- moved U5 113.9 mm to (142.0, 49.4), turned to 270 degrees
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- renumbered H4 to H5, H3 to H6
Connections:
- D4 pad 2: Net-(D4-Pad2) -> (no net)
- J8 pad 6: Net-(J8-Pad6) -> (no net)
- J8 pad 7: Net-(J8-Pad7) -> (no net)
- J9 pad 5: Net-(J9-Pad5) -> Net-(F2-Pad2)
- J9 pad 6: Net-(J9-Pad6) -> Net-(F2-Pad2)
- J9 pad 7: GND -> CycleBTNLED
- J9 pad 8: CycleBTNLED -> SpareBtn1
- Q5 pad 1: Relay_act2 -> (no net)
- Q6 pad 3: +24V -> Net-(D1-Pad1)
- R1 pad 1: +24V -> Net-(D1-Pad1)
- U8 pad 4: SonicGND -> (no net)
- U8 pad 8: Net-(U8-Pad8) -> Sonic24V
Routing:
- net Net-(J7-Pad1): track 0.00 -> 95.0 mm
- net VCC: track 3.06 -> 97.3 mm, vias 0 -> 2
- net Net-(J7-Pad2): track 0.00 -> 89.8 mm
- net Sonic24V: track 0.00 -> 79.0 mm, vias 0 -> 1
- net +5V: track 0.00 -> 71.5 mm, vias 0 -> 1
- net +24V: track 14.3 -> 84.7 mm
- net SonicGND: track 0.00 -> 61.9 mm, vias 0 -> 1
- net Spare1: track 0.00 -> 56.3 mm
- net CycleBTNLEDMCU: track 0.00 -> 53.9 mm, vias 0 -> 1
- net Net-(F2-Pad2): track 0.00 -> 49.3 mm
- net WindowShut: track 0.00 -> 43.0 mm, vias 0 -> 2
- net Beam2: track 0.00 -> 40.6 mm
- net PistonTop: track 0.00 -> 36.9 mm
- net CycleBTNLED: track 0.00 -> 36.0 mm, vias 0 -> 1
- net Beam1: track 0.00 -> 34.8 mm
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Other:
- net class Default: clearance 0.22 -> 0.3; trace_width 0.4 -> 0.6
- net class Small removed
- rule trace_clearance: 0.22 -> 0.3
- rule via_min_drill: 0.3 -> 1.1
- rule via_min_size: 0.4 -> 2

Commit message: layout done
Parts:
- added C10: 100n, Capacitor_SMD:C_0805_2012Metric_Pad1.15x1.40mm_HandSolder, F.Cu at (107.7, 68.1)
- added C9: 100n50V, Capacitor_SMD:C_0805_2012Metric_Pad1.15x1.40mm_HandSolder, F.Cu at (183.4, 96.8)
- added U16: SN74AHCT125N, Package_SO:SOIC-14_3.9x8.7mm_P1.27mm, F.Cu at (110.5, 74.2)
- C1, C5, Q1, Q2, Q3, Q4, Q5, R11, R12, R15, R18, R19, R2, R20, R21, R22, R24, R26, R3, R38, R4, U1: moved to B.Cu
- moved Q1 159.8 mm to (119.6, 69.3), turned to 180 degrees
- moved R7 159.0 mm to (115.6, 87.6), turned to 270 degrees
- moved Q2 157.6 mm to (119.6, 77.2), turned to 180 degrees
- moved Q3 152.2 mm to (119.6, 84.6), turned to 180 degrees
- moved R15 152.1 mm to (130.8, 79.0), turned to 0 degrees
- moved R12 148.3 mm to (130.8, 76.5), turned to 0 degrees
- moved R11 146.2 mm to (130.8, 73.9), turned to 0 degrees
- moved D5 132.7 mm to (112.8, 92.9)
- moved R6 129.3 mm to (112.8, 87.6), turned to 270 degrees
- moved R8 128.4 mm to (118.4, 87.6), turned to 270 degrees
- moved R3 127.2 mm to (146.6, 76.5), turned to 180 degrees
- moved D7 125.1 mm to (118.4, 92.9)
- moved D6 124.5 mm to (115.6, 92.9)
- moved D4 83.5 mm to (152.4, 89.2), turned to 180 degrees
- moved C8 78.0 mm to (153.9, 94.2), turned to 0 degrees
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Connections:
- D4 pad 2: (no net) -> Net-(D4-Pad2)
- J8 pad 6: (no net) -> Net-(J8-Pad6)
- J8 pad 7: (no net) -> Net-(J8-Pad7)
- Q5 pad 1: (no net) -> Net-(Q5-Pad1)
- R6 pad 1: STEP -> Net-(R6-Pad1)
- R7 pad 1: DIR -> Net-(R7-Pad1)
- R8 pad 1: MTR_ENA -> Net-(R8-Pad1)
- REL1 pad 5: (no net) -> Net-(REL1-Pad5)
- REL1 pad 6: (no net) -> Net-(REL1-Pad6)
- REL1 pad 7: (no net) -> Net-(REL1-Pad7)
- REL2 pad 5: (no net) -> Net-(REL2-Pad5)
- REL2 pad 6: (no net) -> Net-(REL2-Pad6)
- REL2 pad 7: (no net) -> Net-(REL2-Pad7)
- U3 pad 1: (no net) -> Net-(U3-Pad1)
- U3 pad 10: (no net) -> Net-(U3-Pad10)
- U3 pad 11: (no net) -> PixelStrip
- U3 pad 12: (no net) -> Net-(U3-Pad12)
- U3 pad 15: (no net) -> Net-(U3-Pad15)
- U3 pad 16: (no net) -> Net-(U3-Pad16)
- U3 pad 2: (no net) -> Net-(U3-Pad2)
- U3 pad 24: Spare1 -> Pixel
- U3 pad 26: Relay_act1 -> Relay_act2
- U3 pad 27: (no net) -> Relay_act1
- U3 pad 28: (no net) -> Net-(U3-Pad28)
- U3 pad 29: (no net) -> Net-(U3-Pad29)
- U3 pad 3: (no net) -> Net-(U3-Pad3)
- U3 pad 30: PixelStrip -> Spare1
- U3 pad 32: Pixel -> Net-(U3-Pad32)
- U3 pad 37: (no net) -> Net-(U3-Pad37)
- U3 pad 38: (no net) -> Net-(U3-Pad38)
- U3 pad 39: (no net) -> Net-(U3-Pad39)
- U3 pad 4: (no net) -> Net-(U3-Pad4)
- U3 pad 8: (no net) -> Net-(U3-Pad8)
- U8 pad 4: (no net) -> SonicGND
Routing:
- net GND: track 11.4 -> 502.7 mm, vias 4 -> 9
- net VCC: track 97.3 -> 285.5 mm, vias 2 -> 3
- net +24V: track 84.7 -> 217.5 mm, vias 1 -> 3
- net Net-(J6-Pad1): track 0.00 -> 125.9 mm, vias 0 -> 2
- net Net-(J6-Pad3): track 0.00 -> 110.8 mm, vias 0 -> 2
- net Estop2: track 0.00 -> 103.1 mm, vias 0 -> 1
- net Net-(J5-Pad2): track 0.00 -> 94.8 mm, vias 0 -> 2
- net Estop1: track 0.00 -> 76.9 mm, vias 0 -> 1
- net SCL: track 4.67 -> 66.6 mm, vias 0 -> 1
- net SDA: track 3.80 -> 49.1 mm, vias 0 -> 1
- net STEP: track 0.00 -> 41.2 mm, vias 0 -> 1
- net +5V: track 71.5 -> 107.8 mm, vias 1 -> 3
- net SonicGND: track 61.9 -> 93.9 mm
- net PixelStrip: track 0.00 -> 31.8 mm
- net Net-(R22-Pad1): track 0.00 -> 28.8 mm
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
Commit message: BOM
Parts:
- U16: value SN74AHCT125N -> 74LVC125
- moved U16 0.14 mm to (110.5, 74.3)
Connections:
- D4 pad 2: Net-(D4-Pad2) -> (no net)
- J8 pad 6: Net-(J8-Pad6) -> (no net)
- J8 pad 7: Net-(J8-Pad7) -> (no net)
- REL1 pad 5: Net-(REL1-Pad5) -> (no net)
- REL1 pad 6: Net-(REL1-Pad6) -> (no net)
- REL1 pad 7: Net-(REL1-Pad7) -> (no net)
- REL2 pad 5: Net-(REL2-Pad5) -> (no net)
- REL2 pad 6: Net-(REL2-Pad6) -> (no net)
- REL2 pad 7: Net-(REL2-Pad7) -> (no net)
- U16 pad 11: Net-(U16-Pad11) -> (no net)
- U16 pad 12: Net-(U16-Pad12) -> (no net)
- U16 pad 13: Net-(U16-Pad13) -> (no net)
- U3 pad 1: Net-(U3-Pad1) -> (no net)
- U3 pad 10: Net-(U3-Pad10) -> (no net)
- U3 pad 12: Net-(U3-Pad12) -> (no net)
- U3 pad 15: Net-(U3-Pad15) -> (no net)
- U3 pad 16: Net-(U3-Pad16) -> (no net)
- U3 pad 2: Net-(U3-Pad2) -> (no net)
- U3 pad 28: Net-(U3-Pad28) -> (no net)
- U3 pad 29: Net-(U3-Pad29) -> (no net)
- U3 pad 3: Net-(U3-Pad3) -> (no net)
- U3 pad 32: Net-(U3-Pad32) -> (no net)
- U3 pad 37: Net-(U3-Pad37) -> (no net)
- U3 pad 38: Net-(U3-Pad38) -> (no net)
- U3 pad 39: Net-(U3-Pad39) -> (no net)
- U3 pad 4: Net-(U3-Pad4) -> (no net)
- U3 pad 8: Net-(U3-Pad8) -> (no net)
Routing:
- net +5V: track 107.8 -> 207.3 mm
- net GND: track 502.7 -> 575.2 mm
- net VCC: track 285.5 -> 346.7 mm
- net Net-(J6-Pad3): track 110.8 -> 105.2 mm
- net WindowShut: track 42.7 -> 37.1 mm
- net Net-(R10-Pad2): track 23.2 -> 26.2 mm
- net DIR: track 20.6 -> 23.5 mm
- net Net-(J5-Pad2): track 94.8 -> 91.9 mm
- net STEP: track 41.2 -> 43.6 mm
- net CycleBTNLED: track 34.2 -> 36.2 mm
- net PistonTop: track 48.8 -> 50.4 mm
- net Net-(R8-Pad1): track 24.9 -> 25.9 mm
- net Spare1: track 52.7 -> 51.8 mm
- net Net-(R36-Pad2): track 28.0 -> 28.8 mm
