File: Ver2/Board/Board.sch (KiCad schematic (older format))
At the start: 76 parts

Commit message: distance beam
Parts:
- removed D?: Green, Diode_SMD:D_0805_2012Metric_Pad1.15x1.40mm_HandSolder, symbol Device:LED_Small_ALT
- removed Q? (x3): A03401, Package_TO_SOT_SMD:SOT-23_Handsoldering, symbol Peters:A03401
- removed R?: 330R, Resistor_SMD:R_0805_2012Metric_Pad1.15x1.40mm_HandSolder, symbol Device:R_Small
- removed R? (x2): 10K, Resistor_SMD:R_0805_2012Metric_Pad1.15x1.40mm_HandSolder, symbol Device:R_Small
- added D? (x3): Green, Diode_SMD:D_0805_2012Metric_Pad1.15x1.40mm_HandSolder, symbol Device:LED_Small_ALT
- added J?: Proximity2, symbol Connector:Screw_Terminal_01x03
- added Q? (x3): BSS138, digikey-footprints:SOT-23-3, symbol dk_Transistors-FETs-MOSFETs-Single:BSS138
- added R? (x4): 10K, Resistor_SMD:R_0805_2012Metric_Pad1.15x1.40mm_HandSolder, symbol Device:R_Small
- added R? (x3): 2K2-10K, Resistor_SMD:R_0805_2012Metric_Pad1.15x1.40mm_HandSolder, symbol Device:R_Small
- added R? (x2): 1K-2K, Resistor_SMD:R_0805_2012Metric_Pad1.15x1.40mm_HandSolder, symbol Device:R_Small
- added U? (x2): PC817, Package_DIP:DIP-4_W7.62mm, symbol Isolator:PC817
- REL? (x2): symbol Peters:IM03GR -> Board-rescue:IM03GR-Peters
- U?: symbol Peters:Bluepill -> Board-rescue:Bluepill-Peters
- U? (x2): symbol dk_Linear-Amplifiers-Instrumentation-OP-Amps-Buffer-Amps:LM358N_LTB -> Board-rescue:LM358N_LTB-dk_Linear-Amplifiers-Instrumentation-OP-Amps-Buffer-Amps
- U?: symbol Peters:AP2210-3.3V -> Board-rescue:AP2210-3.3V-Peters
Connections:
- net labels added: Beam1, Beam2
- net labels removed: SCK
- wire segments 193 -> 205
Other:
- note added: "Doorsafty beam"
- note removed: "Hur gör jag detta?\nTvå kablar till varje switch,\n eller seriekoppla dom i kabinettet?"
- moved on the sheet: J?, R?, U?

Commit message: Layout begun
Parts:
- removed C?: 68uf, Capacitor_SMD:CP_Elec_6.3x5.4, symbol Device:CP
- removed C? (x2): 10uF/50V, Capacitor_SMD:C_2010_5025Metric_Pad1.52x2.65mm_HandSolder, symbol Device:C
- removed C?: 22uF/16V, Capacitor_SMD:C_2010_5025Metric_Pad1.52x2.65mm_HandSolder, symbol Device:C
- removed C?: 10p, Capacitor_SMD:C_0805_2012Metric_Pad1.15x1.40mm_HandSolder, symbol Device:C_Small
- removed D? (x2): Green, Diode_SMD:D_0805_2012Metric_Pad1.15x1.40mm_HandSolder, symbol Device:LED_Small_ALT
- removed J?: LED strip, TerminalBlock:TerminalBlock_bornier-2_P5.08mm, symbol Connector:Screw_Terminal_01x02
- removed J?: Proximity1, symbol Connector:Screw_Terminal_01x03
- removed R?: 2K2-10K, Resistor_SMD:R_0805_2012Metric_Pad1.15x1.40mm_HandSolder, symbol Device:R_Small
- removed R?: 10K, Resistor_SMD:R_0805_2012Metric_Pad1.15x1.40mm_HandSolder, symbol Device:R_Small
- removed U?: V7805-1000, digikey-footprints:3-SIP_Module_V7805-1000, symbol dk_DC-DC-Converters:V7805-1000
- removed U?: AP2210-3.3V, Package_TO_SOT_SMD:SOT-23-5_HandSoldering, symbol Board-rescue:AP2210-3.3V-Peters
- added C1, C2: 10uF/50V, Capacitor_SMD:C_2010_5025Metric_Pad1.52x2.65mm_HandSolder, symbol Device:C
- added C3: 22uF/16V, Capacitor_SMD:C_2010_5025Metric_Pad1.52x2.65mm_HandSolder, symbol Device:C
- added C4: 68uf, Capacitor_SMD:CP_Elec_6.3x5.4, symbol Device:CP
- added C5: 10p, Capacitor_SMD:C_0805_2012Metric_Pad1.15x1.40mm_HandSolder, symbol Device:C_Small
- added J11: Proximity2, TerminalBlock_Phoenix:TerminalBlock_Phoenix_MPT-0,5-3-2.54_1x03_P2.54mm_Horizontal, symbol Connector:Screw_Terminal_01x03
- added J3: Reset_switch, Connector_PinSocket_2.54mm:PinSocket_1x02_P2.54mm_Vertical, symbol Connector:Conn_01x02_Male
- added Q6: A03401-Peters, Package_TO_SOT_SMD:SOT-23_Handsoldering, symbol Board-rescue:A03401-Peters
- added Q7: BSS138, digikey-footprints:SOT-23-3, symbol dk_Transistors-FETs-MOSFETs-Single:BSS138
- added R1, R31, R33, R34: 10K, Resistor_SMD:R_0805_2012Metric_Pad1.15x1.40mm_HandSolder, symbol Device:R_Small
- added R2: 2K2-10K, Resistor_SMD:R_0805_2012Metric_Pad1.15x1.40mm_HandSolder, symbol Device:R_Small
- added R32: 2K, Resistor_SMD:R_0805_2012Metric_Pad1.15x1.40mm_HandSolder, symbol Device:R_Small
- added U1: AP2210-3.3V, Package_TO_SOT_SMD:SOT-23-5_HandSoldering, symbol Board-rescue:AP2210-3.3V-Peters
- added U14: PC817, Package_DIP:DIP-4_W7.62mm, symbol Isolator:PC817
- added U2: V7805-1000, digikey-footprints:3-SIP_Module_V7805-1000, symbol dk_DC-DC-Converters:V7805-1000
- J12, J13, J5, J6: renamed from J?; footprint (none) -> TerminalBlock_Phoenix:TerminalBlock_Phoenix_MPT-0,5-3-2.54_1x03_P2.54mm_Horizontal
- J7: renamed from J?; footprint TerminalBlock:TerminalBlock_bornier-2_P5.08mm -> TerminalBlock_Phoenix:TerminalBlock_Phoenix_MPT-0,5-2-2.54_1x02_P2.54mm_Horizontal
- R29, R30: renamed from R?; value 1K-2K -> 2K
- gave numbers to parts that had none: 66
Connections:
- net labels added: Beam3, CycleBTNLEDMCU
- wire segments 205 -> 225
Other:
- note removed: "LED resistor\nVF=2.2V\n2.2K=9.9mA\n5.1K=4.2mA\n10K=2.2mA"
- moved on the sheet: C6, C7, D3, F1, J1, J10, J12, J13, J2, J7, J8, R10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

Commit message: routing
Parts:
- removed H1, H2, H3, H4: MountingHole, MountingHole:MountingHole_3.2mm_M3, symbol Mechanical:MountingHole
- added D1: 26v, Diode_THT:D_DO-15_P10.16mm_Horizontal, symbol Device:D_Zener_ALT
- added R35: 2K, Resistor_SMD:R_0805_2012Metric_Pad1.15x1.40mm_HandSolder, symbol Device:R_Small
- added R36: 1K-2K, Resistor_SMD:R_0805_2012Metric_Pad1.15x1.40mm_HandSolder, symbol Device:R_Small
- added R37: 10K, Resistor_SMD:R_0805_2012Metric_Pad1.15x1.40mm_HandSolder, symbol Device:R_Small
- added R38: 100R, Resistor_SMD:R_0805_2012Metric_Pad1.15x1.40mm_HandSolder, symbol Device:R_Small
- added U15: PC817, Package_DIP:DIP-4_W7.62mm, symbol Isolator:PC817
- J11, J12, J13, J5, J6: footprint TerminalBlock_Phoenix:TerminalBlock_Phoenix_MPT-0,5-3-2.54_1x03_P2.54mm_Horizontal -> Libs:MKDS1,3-3,81
- J7: footprint TerminalBlock_Phoenix:TerminalBlock_Phoenix_MPT-0,5-2-2.54_1x02_P2.54mm_Horizontal -> TerminalBlock:TerminalBlock_bornier-2_P5.08mm
- REL1, REL2: footprint (none) -> Libs:IM03GR
Connections:
- net labels added: Spare1, SpareBtn1
- wire segments 225 -> 238
Other:
- moved on the sheet: D5, D6, D7, R6, R7, R8

Commit message: layout done
Parts:
- added C10: 100n, Capacitor_SMD:C_0805_2012Metric_Pad1.15x1.40mm_HandSolder, symbol Device:C_Small
- added C9: 100n50V, Capacitor_SMD:C_0805_2012Metric_Pad1.15x1.40mm_HandSolder, symbol Device:C_Small
- added U16: SN74AHCT125N, Package_SO:SOIC-14_3.9x8.7mm_P1.27mm, symbol dk_Logic-Buffers-Drivers-Receivers-Transceivers:SN74AHCT125N
Connections:
- wire segments 238 -> 255
- no-connect marks 0 -> 2
Other:
- moved on the sheet: D1, D5, D6, D7, Q6, Q7, R1, R24, R33, R34, R35, R38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

Commit message: BOM
Parts:
- removed U16: SN74AHCT125N, Package_SO:SOIC-14_3.9x8.7mm_P1.27mm, symbol dk_Logic-Buffers-Drivers-Receivers-Transceivers:SN74AHCT125N
- added U16: 74LVC125, Package_SO:SOIC-14_3.9x8.7mm_P1.27mm, symbol 74xx:74LVC125
Connections:
- wire segments 255 -> 254
Other:
- moved on the sheet: C10, D5, D6, D7, R6, R7, R8
